File: kicad/akohore.kicad_pcb (KiCad board)
At the start: 2 copper layers, 76 parts, among them SW1 SW_SPDT, SW10 SW_Push, SW11 SW_Push, SW12 SW_Push, SW13 SW_Push, SW14 SW_Push, SW15 SW_Push, SW16 SW_Push, SW17 SW_Push, SW18 SW_Push, SW19 SW_Push, SW2 SW_Push, SW20 SW_Push, SW21 SW_Push, SW22 SW_Push, SW23 SW_Push, SW24 SW_Push, SW25 SW_Push, SW26 SW_Push, SW27 SW_Push, SW28 SW_Push, SW29 SW_Push, SW3 SW_Push, SW30 SW_Push, SW31 SW_Push, SW32 SW_Push, SW33 SW_Push, SW34 SW_Push, SW35 SW_Push, SW36 SW_Push, SW37 SW_Push, SW38 SW_Push, SW4 SW_Push, SW5 SW_Push, SW6 SW_Push, SW7 SW_Push, SW8 SW_Push, SW9 SW_Push, U1 ProMicro

Commit message: layout pcb
Parts:
- added SW28: SW_Push, Keebio-Parts:Kailh-PG1350-1u-NoLED, F.Cu at (126.6, -25.7)
- added SW28: SW_Push, Keebio-Parts:Kailh-PG1350-1u-NoLED, B.Cu at (67.4, -25.7)
- added SW29: SW_Push, Keebio-Parts:Kailh-PG1350-1u-NoLED, F.Cu at (144.4, -29.1)
- added SW29: SW_Push, Keebio-Parts:Kailh-PG1350-1u-NoLED, B.Cu at (49.6, -29.2)
- moved SW3 248.2 mm to (-2.25, -55.9), turned to 355 degrees
- moved SW4 242.0 mm to (16.7, -66.5), turned to 355 degrees
- moved SW5 239.4 mm to (35.1, -69.4), turned to 355 degrees
- moved SW14 212.3 mm to (15.3, -49.6), turned to 355 degrees
- moved SW13 208.1 mm to (-3.73, -39.0), turned to 355 degrees
- moved SW9 203.4 mm to (141.4, -62.9), turned to 5 degrees
- moved SW6 198.8 mm to (52.6, -63.0), turned to 355 degrees
- moved SW19 193.5 mm to (142.9, -45.9), turned to 5 degrees
- moved SW29 193.0 mm to (144.4, -29.0), turned to 5 degrees
- moved SW15 189.6 mm to (33.6, -52.5), turned to 355 degrees
- moved SW7 188.5 mm to (70.3, -59.6), turned to 355 degrees
- moved SW24 181.8 mm to (13.8, -32.7), turned to 355 degrees
- moved SW8 181.5 mm to (123.7, -59.4), turned to 5 degrees
- moved SW32 177.6 mm to (199.2, -21.9), turned to 5 degrees
- moved SW23 171.1 mm to (-5.21, -22.0), turned to 355 degrees
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
Commit message: add diodes
Parts:
- removed the SW28 at (126.6, -25.7)
- removed the SW28 at (67.4, -25.7)
- removed the SW28 at (126.6, -25.6)
- removed the SW29 at (144.4, -29.1)
- removed the SW29 at (49.6, -29.2)
- removed the SW29 at (144.4, -29.0)
- added SW28: SW_Push, custom-parts:customchocfootprint, F.Cu at (62.6, -28.5)
- added SW29: SW_Push, custom-parts:customchocfootprint, F.Cu at (80.4, -32.0)
- SW10, SW11, SW12, SW13, SW14, SW15, SW16, SW17, SW18, SW19, SW20, SW21, SW22, SW23, SW24, SW25, SW26, SW27, SW3, SW30, SW31, SW32, SW33, SW34, SW35, SW36, SW37, SW38, SW4, SW5, SW6, SW7, SW8, SW9: footprint Keebio-Parts:Kailh-PG1350-1u-NoLED -> custom-parts:customchocfootprint
- moved SW1 332.3 mm to (70.2, -180.2), turned to 180 degrees
- moved D11 326.3 mm to (-85.1, -47.8), turned to 355 degrees
- moved D1 323.5 mm to (-83.6, -64.7), turned to 355 degrees
- moved D21 322.2 mm to (-86.6, -30.8), turned to 355 degrees
- moved D2 313.3 mm to (-64.6, -75.3), turned to 355 degrees
- moved D12 310.1 mm to (-66.1, -58.4), turned to 355 degrees
- moved D3 309.1 mm to (-46.3, -78.2), turned to 355 degrees
- moved D13 294.2 mm to (-47.8, -61.3), turned to 355 degrees
- moved D22 290.6 mm to (-67.6, -41.5), turned to 355 degrees
- moved D23 290.3 mm to (-49.2, -44.3), turned to 355 degrees
- moved D4 288.2 mm to (-28.8, -71.8), turned to 355 degrees
- moved D5 273.9 mm to (-11.0, -68.4), turned to 355 degrees
- moved SW2 270.5 mm to (62.9, -169.6), turned to 90 degrees
- moved D14 266.7 mm to (-30.3, -54.9), turned to 355 degrees
- moved D24 264.1 mm to (-31.8, -37.9), turned to 355 degrees
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
Commit message: last commit before edgecuts
Parts:
- moved BT1 223.0 mm to (33.3, -38.1)
- moved SW2 115.4 mm to (11.6, -66.3), turned to 180 degrees
- moved SW1 112.5 mm to (38.1, -72.4), turned to 0 degrees
- moved U1 108.8 mm to (25.4, -61.0)
- moved D8 6.18 mm to (93.5, -84.0)
- moved SW10 6.18 mm to (95.9, -78.3)
- moved D18 6.18 mm to (94.9, -67.0)
- moved D19 6.18 mm to (113.3, -64.1)
- moved D20 6.18 mm to (132.3, -53.5)
- moved D26 6.18 mm to (61.2, -40.3)
- moved D9 6.18 mm to (111.8, -81.1)
- moved SW21 6.18 mm to (115.7, -58.5)
- moved SW8 6.18 mm to (60.6, -68.5)
- moved SW28 6.18 mm to (63.6, -34.6)
- moved D30 6.18 mm to (133.7, -36.6)
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
Commit message: nvm, not the last one
Parts:
- moved BT1 11.2 mm to (23.0, -42.4)
Changed lines of the file:
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@@
   )
   (module Connector_Wire:battery (layer F.Cu)
-    (at 33.3 -38.1)
+    (at 23.013 -42.418)
     (descr "Soldered wire connection, for 2 times 0.5 mm² wires, reinforced insulation, conductor diameter 0.9mm, outer diameter 2.3mm, size source Multi-Contact FLEXI-xV 0.5 (https://ec.staubli.com/AcroFiles/Catalogues/TM_Cab-Main-11014119_(en)_hi.pdf), bend radius 3 times outer diameter, generated with kicad-footprint-generator")
     (tags "connector wire 0.5sqmm")

Commit message: routing half
Parts:
- moved SW2 21.2 mm to (13.8, -87.4)
- moved U1 14.6 mm to (25.4, -75.6)
- moved SW1 7.69 mm to (39.5, -80.0)
- moved D7 3.83 mm to (76.0, -77.1)
- moved SW29 0.37 mm to (81.0, -38.0)
- moved D20 0.37 mm to (132.0, -53.4)
- moved D35 0.37 mm to (70.7, -23.0)
- moved D8 0.37 mm to (93.1, -83.8)
- moved SW18 0.37 mm to (61.8, -51.4)
- moved SW38 0.37 mm to (93.5, -22.0)
- moved SW22 0.37 mm to (134.3, -47.8)
- moved D27 0.37 mm to (78.6, -43.6)
- moved D36 0.37 mm to (90.6, -27.4)
- moved SW21 0.37 mm to (115.3, -58.4)
- moved D34 0.37 mm to (51.3, -15.7)
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Connections:
- SW1 pad 2: Net-(SW1-Pad2) -> +BATT
- SW19 pad 2: Net-(SW19-Pad2) -> COL6
- SW29 pad 1: (no net) -> Net-(D27-Pad2)
- SW29 pad 2: (no net) -> COL6
- SW9 pad 2: Net-(SW9-Pad2) -> COL6
Routing:
- net ROW0: track 0.00 -> 78.4 mm
- net ROW2: track 0.00 -> 76.7 mm
- net ROW1: track 0.00 -> 75.7 mm
- net COL5: track 0.00 -> 69.4 mm
- net COL6: track 0.00 -> 65.1 mm
- net COL7: track 0.00 -> 64.9 mm
- net ROW3: track 0.00 -> 41.3 mm
- net COL8: track 0.00 -> 37.6 mm
- net COL9: track 0.00 -> 37.6 mm
- net Net-(D17-Pad2): track 0.00 -> 13.7 mm
- net Net-(D10-Pad2): track 0.00 -> 13.6 mm
- net Net-(D29-Pad2): track 0.00 -> 13.6 mm
- net Net-(D19-Pad2): track 0.00 -> 13.6 mm
- net Net-(D36-Pad2): track 0.00 -> 13.5 mm
- net Net-(D30-Pad2): track 0.00 -> 13.5 mm
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Other:
- board outline added: 248.2 x 100 mm
- net class Default: clearance 0.2 -> 0.5
- net class Power added: clearance 0.5, trace_width 0.4, via_dia 0.8, via_drill 0.4
- rule trace_clearance: 0.2 -> 0.5

Commit message: readyforfirstcheck
Parts:
- moved SW1 28.8 mm to (13.6, -92.5)
- moved SW2 27.2 mm to (-13.3, -85.7)
- moved D10 25.9 mm to (104.6, -71.7)
- moved D18 25.9 mm to (68.8, -68.3)
- moved D29 25.9 mm to (88.6, -48.5)
- moved D30 25.9 mm to (107.6, -37.8)
- moved D7 25.9 mm to (50.2, -78.5)
- moved D8 25.9 mm to (67.3, -85.2)
- moved D9 25.9 mm to (85.6, -82.4)
- moved SW10 25.9 mm to (69.7, -79.6)
- moved SW11 25.9 mm to (88.0, -76.7)
- moved SW12 25.9 mm to (107.0, -66.1)
- moved SW32 25.9 mm to (110.0, -32.2)
- moved SW38 25.9 mm to (67.6, -23.4)
- moved SW9 25.9 mm to (52.2, -73.2)
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
Commit message: finished, no checks yet
Parts:
- moved D9 3.25 mm to (86.7, -85.4)
- moved D29 2.49 mm to (89.7, -50.7)
- moved SW10 2.49 mm to (70.9, -81.8)
- moved SW22 2.49 mm to (109.7, -51.4)
- moved D16 2.49 mm to (34.7, -60.6)
- moved D7 2.49 mm to (51.3, -80.8)
- moved SW28 2.49 mm to (38.5, -38.1)
- moved SW9 2.49 mm to (53.3, -75.4)
- moved SW38 2.49 mm to (68.8, -25.6)
- moved D34 2.49 mm to (26.6, -19.3)
- moved D35 2.49 mm to (46.0, -26.6)
- moved D10 2.49 mm to (105.8, -73.9)
- moved D18 2.49 mm to (69.9, -70.5)
- moved D19 2.49 mm to (88.3, -67.6)
- moved D20 2.49 mm to (107.3, -57.0)
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Routing:
- net ROW0: track 78.4 -> 287.5 mm
- net ROW1: track 75.7 -> 253.5 mm
- net ROW2: track 76.7 -> 253.4 mm
- net COL9: track 37.6 -> 207.2 mm
- net COL0: track 0.00 -> 159.1 mm
- net COL2: track 0.00 -> 148.3 mm
- net ROW3: track 41.3 -> 188.3 mm, vias 0 -> 1
- net COL8: track 37.6 -> 180.6 mm
- net COL1: track 0.00 -> 139.9 mm
- net COL3: track 0.00 -> 122.4 mm
- net COL7: track 64.9 -> 181.1 mm
- net COL4: track 0.00 -> 112.3 mm
- net COL6: track 65.1 -> 153.5 mm
- net GND: track 1.24 -> 81.9 mm
- net Net-(BT1-Pad1): track 0.00 -> 66.1 mm
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