File: kicad/akohore.kicad_pcb (KiCad board)
At the start: 2 copper layers, 248.2 x 100 mm, 76 parts, among them SW1 SW_SPDT, SW10 SW_Push, SW11 SW_Push, SW12 SW_Push, SW13 SW_Push, SW14 SW_Push, SW15 SW_Push, SW16 SW_Push, SW17 SW_Push, SW18 SW_Push, SW19 SW_Push, SW2 SW_Push, SW20 SW_Push, SW21 SW_Push, SW22 SW_Push, SW23 SW_Push, SW24 SW_Push, SW25 SW_Push, SW26 SW_Push, SW27 SW_Push, SW28 SW_Push, SW29 SW_Push, SW3 SW_Push, SW30 SW_Push, SW31 SW_Push, SW32 SW_Push, SW33 SW_Push, SW34 SW_Push, SW35 SW_Push, SW36 SW_Push, SW37 SW_Push, SW38 SW_Push, SW4 SW_Push, SW5 SW_Push, SW6 SW_Push, SW7 SW_Push, SW8 SW_Push, SW9 SW_Push, U1 ProMicro

Commit message: production pcb files, silk and mounting holes add
Parts:
- added G***: LOGO, custom-parts:astro, B.Cu at (0.33, -17.6)
- added G***: LOGO, custom-parts:logo6, F.Cu at (0.33, -10.6)
- added G***: LOGO, custom-parts:logocopper, F.Cu at (0.33, -10.6)
- added REF**: MountingHole_2.2mm_M2_Pad, MountingHole:MountingHole_2.2mm_M2_Pad, F.Cu at (-19.7, -70.5)
- added REF**: MountingHole_2.2mm_M2_Pad, MountingHole:MountingHole_2.2mm_M2_Pad, F.Cu at (20.3, -70.5)
- added REF**: MountingHole_2.2mm_M2_Pad, MountingHole:MountingHole_2.2mm_M2_Pad, F.Cu at (20.3, -30.6)
- added REF**: MountingHole_2.2mm_M2_Pad, MountingHole:MountingHole_2.2mm_M2_Pad, F.Cu at (-19.7, -30.6)
- added REF**: MountingHole_2.2mm_M2_Pad, MountingHole:MountingHole_2.2mm_M2_Pad, F.Cu at (90.3, -20.6)
- added REF**: MountingHole_2.2mm_M2_Pad, MountingHole:MountingHole_2.2mm_M2_Pad, F.Cu at (-89.7, -20.6)
- added REF**: MountingHole_2.2mm_M2_Pad, MountingHole:MountingHole_2.2mm_M2_Pad, F.Cu at (-109.7, -85.5)
- added REF**: MountingHole_2.2mm_M2_Pad, MountingHole:MountingHole_2.2mm_M2_Pad, F.Cu at (110.3, -85.5)
- moved BT1 9.53 mm to (-1.98, -53.0)
Routing:
- net Net-(BT1-Pad1): track 66.1 -> 52.6 mm
- net GND: track 81.9 -> 72.4 mm
- net (no net): track 0.96 -> 0.00 mm
Other:
- board text added: "Licensed under CERN-OHL-P v2."
- board text added: "designed alongside Bonsa"
- board text added: "powered by ZMK"
- board text added: "thank you everyone for the help"
