File: kicad/ahokore.kicad_pcb (KiCad board)
At the start: 2 copper layers, 248.2 x 100 mm, 87 parts, among them SW1 SW_SPDT, SW10 SW_Push, SW11 SW_Push, SW12 SW_Push, SW13 SW_Push, SW14 SW_Push, SW15 SW_Push, SW16 SW_Push, SW17 SW_Push, SW18 SW_Push, SW19 SW_Push, SW2 SW_Push, SW20 SW_Push, SW21 SW_Push, SW22 SW_Push, SW23 SW_Push, SW24 SW_Push, SW25 SW_Push, SW26 SW_Push, SW27 SW_Push, SW28 SW_Push, SW29 SW_Push, SW3 SW_Push, SW30 SW_Push, SW31 SW_Push, SW32 SW_Push, SW33 SW_Push, SW34 SW_Push, SW35 SW_Push, SW36 SW_Push, SW37 SW_Push, SW38 SW_Push, SW4 SW_Push, SW5 SW_Push, SW6 SW_Push, SW7 SW_Push, SW8 SW_Push, SW9 SW_Push, U1 ProMicro

Commit message: i forgot to save before updates
Routing:
- net Net-(D9-Pad2): track 13.4 -> 14.2 mm
Other:
- board text added: "Ahokore V1"
Changed lines of the file:
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@@
   (general
     (thickness 1.6)
-    (drawings 15)
-    (tracks 488)
+    (drawings 16)
+    (tracks 489)
     (zones 0)
     (modules 87)
@@
     )
   )
+  (gr_text "Ahokore V1" (at 0.325 -57.05) (layer B.SilkS)
+    (effects (font (size 2 2) (thickness 0.3)) (justify mirror))
+  )
   (gr_text "Licensed under CERN-OHL-P v2." (at 0.325 -37.05) (layer B.SilkS)
     (effects (font (size 2 2) (thickness 0.3)) (justify mirror))
@@
   (segment (start 84.244943 -85.181886) (end 84.288521 -84.683789) (width 0.25) (layer B.Cu) (net 12))
   (segment (start 87.17953 -75.035547) (end 89.454494 -73.126626) (width 0.25) (layer B.Cu) (net 12))
+  (segment (start 84.288521 -84.683789) (end 84.288521 -83.863789) (width 0.25) (layer B.Cu) (net 12))
   (segment (start 105.573305 -71.320582) (end 106.159605 -64.619132) (width 0.25) (layer B.Cu) (net 13))
   (segment (start 103.33852 -73.195789) (end 105.573305 -71.320582) (width 0.25) (layer B.Cu) (net 13))
