File: v1.1/ahokore.kicad_pcb (KiCad board)
At the start: 2 copper layers, 248.2 x 100 mm, 87 parts, among them SW1 SW_SPDT, SW10 SW_Push, SW11 SW_Push, SW12 SW_Push, SW13 SW_Push, SW14 SW_Push, SW15 SW_Push, SW16 SW_Push, SW17 SW_Push, SW18 SW_Push, SW19 SW_Push, SW2 SW_Push, SW20 SW_Push, SW21 SW_Push, SW22 SW_Push, SW23 SW_Push, SW24 SW_Push, SW25 SW_Push, SW26 SW_Push, SW27 SW_Push, SW28 SW_Push, SW29 SW_Push, SW3 SW_Push, SW30 SW_Push, SW31 SW_Push, SW32 SW_Push, SW33 SW_Push, SW34 SW_Push, SW35 SW_Push, SW36 SW_Push, SW37 SW_Push, SW38 SW_Push, SW4 SW_Push, SW5 SW_Push, SW6 SW_Push, SW7 SW_Push, SW8 SW_Push, SW9 SW_Push, U1 ProMicro

Commit message: wooohoooo
Parts:
- removed G***: LOGO, custom-parts:astro
- removed G***: LOGO, custom-parts:logo6
- removed G***: LOGO, custom-parts:logocopper
- removed REF** (x8): MountingHole_2.2mm_M2_Pad, MountingHole:MountingHole_2.2mm_M2_Pad
- added BT2: Battery_Cell, Connector_JST:JST_PH_S2B-PH-SM4-TB_1x02-1MP_P2.00mm_Horizontal, F.Cu at (20.3, -70.5)
- BT1: footprint Connector_Wire:battery -> Connector_Wire:SolderWire-0.75sqmm_1x02_P7mm_D1.25mm_OD3.5mm
- SW10, SW11, SW12, SW13, SW14, SW15, SW16, SW17, SW18, SW19, SW20, SW21, SW22, SW23, SW24, SW25, SW26, SW27, SW28, SW29, SW3, SW30, SW31, SW32, SW33, SW34, SW35, SW36, SW37, SW38, SW4, SW5, SW6, SW7, SW8, SW9: footprint custom-parts:customchocfootprint -> switchfootprints:Choc_PG1350_Choc_Spacing
- moved D1 322.9 mm to (199.4, 21.5), turned to 0 degrees
- moved D2 320.4 mm to (218.5, 1.83), turned to 0 degrees
- moved D12 315.6 mm to (218.5, -8.85), turned to 0 degrees
- moved D11 305.6 mm to (180.3, 37.0), turned to 0 degrees
- moved D3 274.9 mm to (160.2, 60.4), turned to 0 degrees
- moved D15 270.4 mm to (229.1, -17.4), turned to 0 degrees
- moved D5 266.3 mm to (218.5, -0.84), turned to 0 degrees
- moved D13 261.3 mm to (155.8, 55.1), turned to 0 degrees
- moved D21 260.2 mm to (129.0, 57.8), turned to 0 degrees
- moved D4 255.5 mm to (160.2, 57.8), turned to 0 degrees
- moved D22 251.4 mm to (135.0, 55.1), turned to 0 degrees
- moved D14 240.4 mm to (149.8, 60.4), turned to 0 degrees
- moved D23 227.1 mm to (124.6, 55.1), turned to 0 degrees
- moved D24 206.2 mm to (118.6, 60.4), turned to 0 degrees
- moved D6 192.2 mm to (199.4, 18.8), turned to 0 degrees
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Connections:
- U1 pad 3: Net-(U1-Pad3) -> GND
- U1 pad 4: Net-(U1-Pad4) -> GND
Routing:
- net ROW0: track 287.5 -> 0.00 mm
- net ROW1: track 253.5 -> 0.00 mm
- net ROW2: track 253.4 -> 0.00 mm
- net COL9: track 207.2 -> 0.00 mm
- net ROW3: track 188.3 -> 0.00 mm, vias 1 -> 0
- net COL7: track 181.1 -> 0.00 mm
- net COL8: track 180.6 -> 0.00 mm
- net COL0: track 159.1 -> 0.00 mm
- net COL6: track 153.5 -> 0.00 mm
- net COL2: track 148.3 -> 0.00 mm
- net COL1: track 139.9 -> 0.00 mm
- net COL5: track 129.8 -> 0.00 mm
- net COL3: track 122.4 -> 0.00 mm
- net COL4: track 112.3 -> 0.00 mm
- net GND: track 72.4 -> 0.00 mm
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Other:
- board outline removed
- board text removed: "Ahokore V1"
- board text removed: "Licensed under CERN-OHL-P v2."
- board text removed: "designed alongside Bonsa"
- board text removed: "powered by ZMK"
- board text removed: "thank you everyone for the help"
