File: v2/pcbfiles/ahokore.kicad_pcb (KiCad board)
At the start: 2 copper layers, 265.7 x 104.1 mm, 98 parts, among them J1 Conn_01x04_Female, Q1 AO3401A, SW1 SW_SPST, SW10 SW_Push, SW11 SW_Push, SW12 SW_Push, SW13 SW_Push, SW14 SW_Push, SW15 SW_Push, SW16 SW_Push, SW17 SW_Push, SW18 SW_Push, SW19 SW_Push, SW2 SW_Push, SW20 SW_Push, SW21 SW_Push, SW22 SW_Push, SW23 SW_Push, SW24 SW_Push, SW25 SW_Push, SW26 SW_Push, SW27 SW_Push, SW28 SW_Push, SW29 SW_Push, SW3 SW_Push, SW30 SW_Push, SW31 SW_Push, SW32 SW_Push, SW33 SW_Push, SW34 SW_Push, SW35 SW_Push, SW36 SW_Push, SW37 SW_Push, SW38 SW_SPDT, SW4 SW_Push, SW5 SW_Push, SW6 SW_Push, SW7 SW_Push, SW8 SW_Push, SW9 SW_Push, U2 AP2112K-3.3, U3 TP4054, U4 nRF52840_holyiot_18010

Commit message: production
Parts:
- added C3: 1uF, Capacitor_SMD:C_0805_2012Metric, F.Cu at (148.0, 32.5)
- added C4: 1uF, Capacitor_SMD:C_0805_2012Metric, F.Cu at (152.2, 32.5)
- added G***: LOGO, custom-parts:fe4, F.Cu at (152.0, 98.7)
- added G***: LOGO, custom-parts:v2-2, F.Cu at (143.8, 94.2)
- added G***: LOGO, custom-parts:dezli, F.Cu at (114.2, 94.2)
- added G***: LOGO, custom-parts:ahokore3, F.Cu at (112.0, 98.2)
- added G***: LOGO, custom-parts:fantail3, B.Cu at (130.0, 57.0)
- BT1: footprint Connector_JST:JST_PH_S2B-PH-SM4-TB_1x02-1MP_P2.00mm_Horizontal -> custom-parts:JST_PH_S2B-PH-K_1x02_P2.00mm_Horizontal
- moved R7 5.01 mm to (148.0, 42.3)
- moved R8 5.01 mm to (152.2, 42.3)
- moved D1 5.00 mm to (152.2, 37.5)
- moved Q1 5.00 mm to (148.0, 37.5)
- moved BT1 0.40 mm to (130.0, 26.4)
Connections:
- SW38 pad : (no net) -> Earth
- SW38 pad 0: (no net) -> Earth
Routing:
- net VBUS: track 142.1 -> 154.3 mm
- net (no net): track 9.13 -> 0.00 mm
- net Earth: track 56.4 -> 65.6 mm
- net VDD_NRF: track 66.7 -> 75.5 mm, vias 2 -> 3
- net BVOLT: track 57.7 -> 50.8 mm
- net Net-(C4-Pad1): track 11.1 -> 16.8 mm
- net VBAT: track 49.3 -> 46.6 mm, vias 2 -> 3
- net GND: track 39.6 -> 38.4 mm
Other:
- board text added: "JLCJLCJLCJLC"
