File: v2/pcbfiles/ahokore.sch (KiCad schematic (older format))
At the start: 99 parts, among them J1 Conn_01x04_Female, Q1 AO3401A, SW1 SW_SPST, SW10 SW_Push, SW11 SW_Push, SW12 SW_Push, SW13 SW_Push, SW14 SW_Push, SW15 SW_Push, SW16 SW_Push, SW17 SW_Push, SW18 SW_Push, SW19 SW_Push, SW2 SW_Push, SW20 SW_Push, SW21 SW_Push, SW22 SW_Push, SW23 SW_Push, SW24 SW_Push, SW25 SW_Push, SW26 SW_Push, SW27 SW_Push, SW28 SW_Push, SW29 SW_Push, SW3 SW_Push, SW30 SW_Push, SW31 SW_Push, SW32 SW_Push, SW33 SW_Push, SW34 SW_Push, SW35 SW_Push, SW36 SW_Push, SW37 SW_Push, SW38 SW_SPDT, SW4 SW_Push, SW5 SW_Push, SW6 SW_Push, SW7 SW_Push, SW8 SW_Push, SW9 SW_Push, U2 AP2112K-3.3, U3 TP4054, U4 nRF52840_holyiot_18010

Commit message: production
Parts:
- added C3, C4: 1uF, Capacitor_SMD:C_0805_2012Metric, symbol Device:C_Small
- BT1: footprint Connector_JST:JST_PH_S2B-PH-SM4-TB_1x02-1MP_P2.00mm_Horizontal -> custom-parts:JST_PH_S2B-PH-K_1x02_P2.00mm_Horizontal
Connections:
- net GND: now also C3.2, C4.2
- net VDD_NRF: now also C3.1
- net at D1.1 (K), Q1.2 (S), U2.1 (VIN)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: now also C4.1
Changed lines of the file:
@@
 	1    0    0    -1
 $EndComp
-Text GLabel 8000 1550 2    50   Input ~ 0
+Text GLabel 8350 1550 2    50   Input ~ 0
 VDD_NRF
 $Comp
@@
 	7100 1400 7100 1450
 Connection ~ 7100 1450
-Wire Wire Line
-	7100 1450 7400 1450
 Text GLabel 1100 6300 3    50   Input ~ 0
 VDD_NRF
@@
 F 0 "BT1" V 3195 7050 50  0000 C CNN
 F 1 "Battery_Cell" V 3286 7050 50  0000 C CNN
-F 2 "Connector_JST:JST_PH_S2B-PH-SM4-TB_1x02-1MP_P2.00mm_Horizontal" V 3450 7060 50  0001 C CNN
+F 2 "custom-parts:JST_PH_S2B-PH-K_1x02_P2.00mm_Horizontal" V 3450 7060 50  0001 C CNN
 F 3 "~" V 3450 7060 50  0001 C CNN
 	1    3450 7000
@@
 Text GLabel 2300 5500 2    50   Input ~ 0
 ROW2
+Wire Wire Line
+	7100 1450 7250 1450
+$Comp
+L Device:C_Small C4
+U 1 1 60317035
+P 7050 1750
+F 0 "C4" H 7142 1796 50  0000 L CNN
+F 1 "1uF" H 7142 1705 50  0000 L CNN
+F 2 "Capacitor_SMD:C_0805_2012Metric" H 7050 1750 50  0001 C CNN
+F 3 "~" H 7050 1750 50  0001 C CNN
+	1    7050 1750
+	1    0    0    -1
+$EndComp
+Wire Wire Line
+	7050 1650 7250 1650
+Wire Wire Line
+	7250 1650 7250 1450
+Connection ~ 7250 1450
+Wire Wire Line
+	7250 1450 7400 1450
+Wire Wire Line
+	7050 1850 7050 1950
+$Comp
+L power:GND #PWR0103
+U 1 1 6032FF88
+P 7050 1950
+F 0 "#PWR0103" H 7050 1700 50  0001 C CNN
+F 1 "GND" H 7055 1777 50  0000 C CNN
+F 2 "" H 7050 1950 50  0001 C CNN
+F 3 "" H 7050 1950 50  0001 C CNN
+	1    7050 1950
+	1    0    0    -1
+$EndComp
+$Comp
+L Device:C_Small C3
+U 1 1 60332105
+P 8100 1650
+F 0 "C3" H 8192 1696 50  0000 L CNN
+F 1 "1uF" H 8192 1605 50  0000 L CNN
+F 2 "Capacitor_SMD:C_0805_2012Metric" H 8100 1650 50  0001 C CNN
+F 3 "~" H 8100 1650 50  0001 C CNN
+	1    8100 1650
+	1    0    0    -1
+$EndComp
+Wire Wire Line
+	8100 1750 8100 1850
+$Comp
+L power:GND #PWR0104
+U 1 1 6033210C
+P 8100 1850
+F 0 "#PWR0104" H 8100 1600 50  0001 C CNN
+F 1 "GND" H 8105 1677 50  0000 C CNN
+F 2 "" H 8100 1850 50  0001 C CNN
+F 3 "" H 8100 1850 50  0001 C CNN
+	1    8100 1850
+	1    0    0    -1
+$EndComp
+Wire Wire Line
+	8000 1550 8100 1550
+Connection ~ 8100 1550
+Wire Wire Line
+	8100 1550 8350 1550
 $EndSCHEMATC
